File: kicad-tut.kicad_pcb (KiCad board)
At the start: 2 copper layers, 45.7 x 33 mm, 7 parts, among them J1 MYCONN3, U1 PIC12C508A-ISN

Commit message: Made final changes to the board design and added screenshots of the board.
Signed-off-by: Suyash <in.suyash@gmail.com>
Other:
- board text added: "Blinky Board KiCad"
Changed lines of the file:
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@@
   (general
     (thickness 1.6)
-    (drawings 7)
+    (drawings 8)
     (tracks 36)
     (zones 0)
@@
     (pad 2 thru_hole circle (at 0 0) (size 7 7) (drill 3.5) (layers *.Cu *.Mask Dwgs.User))
   )
+  (gr_text "Blinky Board\nKiCad" (at 128.524 80.772) (layer F.SilkS)
+    (effects (font (size 1.5 1.5) (thickness 0.3)))
+  )
   (gr_text "v1.0\n" (at 162.56 79.502) (layer B.Cu)
