File: kicad-tut.sch (KiCad schematic (older format))
At the start: 5 parts

Commit message: completed board routing
Parts:
- D1: renamed from D?; footprint (none) -> LED_THT:LED_D5.0mm
- J1: renamed from J?; footprint (none) -> Connector:Banana_Jack_3Pin
- R1, R2: renamed from R?; footprint (none) -> Resistor_THT:R_Axial_DIN0204_L3.6mm_D1.6mm_P7.62mm_Horizontal
- gave numbers to parts that had none: 1
Connections:
- net labels added: LEDtoR, uCtoLED
- wire segments 12 -> 16
- no-connect marks 0 -> 4
Other:
- note added: "Needed to supress KiCad DRC warning.\n"
Changed lines of the file:
@@
 EESchema Schematic File Version 4
+LIBS:kicad-tut-cache
 EELAYER 26 0
 EELAYER END
@@
 Title "KiCad Tutorial"
 Date "2019-09-09"
-Rev ""
+Rev "v1.0"
 Comp ""
 Comment1 ""
@@
 $EndBitmap
 $Comp
-L microchip_pic12mcu:PIC12C508A-ISN U?
+L microchip_pic12mcu:PIC12C508A-ISN U1
 U 1 1 5D761873
 P 5700 4100
-F 0 "U?" H 6050 4600 50  0000 C CNN
+F 0 "U1" H 6050 4600 50  0000 C CNN
 F 1 "PIC12C508A-ISN" H 5300 4600 50  0000 C CNN
 F 2 "Package_DIP:DIP-8_W7.62mm" H 6300 4750 50  0001 C CNN
@@
 $EndComp
 $Comp
-L Device:LED D?
+L Device:LED D1
 U 1 1 5D761962
 P 6700 3750
-F 0 "D?" H 6691 3966 50  0000 C CNN
+F 0 "D1" H 6691 3966 50  0000 C CNN
 F 1 "LED" H 6691 3875 50  0000 C CNN
-F 2 "" H 6700 3750 50  0001 C CNN
+F 2 "LED_THT:LED_D5.0mm" H 6700 3750 50  0001 C CNN
 F 3 "~" H 6700 3750 50  0001 C CNN
 	1    6700 3750
@@
 $EndComp
 $Comp
-L myLib:MYCONN3 J?
+L myLib:MYCONN3 J1
 U 1 1 5D761E83
 P 6850 4500
-F 0 "J?" H 6856 4825 50  0000 C CNN
+F 0 "J1" H 6856 4825 50  0000 C CNN
 F 1 "MYCONN3" H 6856 4734 50  0000 C CNN
-F 2 "" H 6950 4500 50  0001 C CNN
+F 2 "Connector:Banana_Jack_3Pin" H 6950 4500 50  0001 C CNN
 F 3 "" H 6950 4500 50  0001 C CNN
 	1    6850 4500
@@
 $EndComp
 $Comp
-L power:VCC #PWR?
+L power:VCC #PWR01
 U 1 1 5D761F83
 P 5700 3400
-F 0 "#PWR?" H 5700 3250 50  0001 C CNN
+F 0 "#PWR01" H 5700 3250 50  0001 C CNN
 F 1 "VCC" H 5717 3573 50  0000 C CNN
 F 2 "" H 5700 3400 50  0001 C CNN
@@
 $EndComp
 $Comp
-L power:GND #PWR?
+L power:GND #PWR02
 U 1 1 5D761FCE
 P 5700 4800
-F 0 "#PWR?" H 5700 4550 50  0001 C CNN
+F 0 "#PWR02" H 5700 4550 50  0001 C CNN
 F 1 "GND" H 5705 4627 50  0000 C CNN
 F 2 "" H 5700 4800 50  0001 C CNN
@@
 $EndComp
 $Comp
-L Device:R R?
+L Device:R R1
 U 1 1 5D762095
 P 7200 3750
-F 0 "R?" V 7300 3700 50  0000 L CNN
+F 0 "R1" V 7300 3700 50  0000 L CNN
 F 1 "1 k" V 7100 3700 50  0000 L CNN
-F 2 "" V 7130 3750 50  0001 C CNN
+F 2 "Resistor_THT:R_Axial_DIN0204_L3.6mm_D1.6mm_P7.62mm_Horizontal" V 7130 3750 50  0001 C CNN
 F 3 "~" H 7200 3750 50  0001 C CNN
 	1    7200 3750
@@
 $EndComp
 $Comp
-L power:VCC #PWR?
+L power:VCC #PWR05
 U 1 1 5D76212F
 P 7400 3550
-F 0 "#PWR?" H 7400 3400 50  0001 C CNN
+F 0 "#PWR05" H 7400 3400 50  0001 C CNN
 F 1 "VCC" H 7417 3723 50  0000 C CNN
 F 2 "" H 7400 3550 50  0001 C CNN
@@
 $EndComp
 $Comp
-L Device:R R?
+L Device:R R2
 U 1 1 5D7624C6
 P 7350 4500
-F 0 "R?" V 7450 4450 50  0000 L CNN
+F 0 "R2" V 7450 4450 50  0000 L CNN
 F 1 "100R" V 7250 4450 50  0000 L CNN
-F 2 "" V 7280 4500 50  0001 C CNN
+F 2 "Resistor_THT:R_Axial_DIN0204_L3.6mm_D1.6mm_P7.62mm_Horizontal" V 7280 4500 50  0001 C CNN
 F 3 "~" H 7350 4500 50  0001 C CNN
 	1    7350 4500
@@
 	7400 3750 7400 3550
 $Comp
-L power:VCC #PWR?
+L power:VCC #PWR03
 U 1 1 5D7625C1
 P 7150 4250
-F 0 "#PWR?" H 7150 4100 50  0001 C CNN
+F 0 "#PWR03" H 7150 4100 50  0001 C CNN
 F 1 "VCC" H 7167 4423 50  0000 C CNN
 F 2 "" H 7150 4250 50  0001 C CNN
@@
 $EndComp
 $Comp
-L power:GND #PWR?
+L power:GND #PWR04
 U 1 1 5D762617
 P 7150 4700
-F 0 "#PWR?" H 7150 4450 50  0001 C CNN
+F 0 "#PWR04" H 7150 4450 50  0001 C CNN
 F 1 "GND" H 7155 4527 50  0000 C CNN
 F 2 "" H 7150 4700 50  0001 C CNN
@@
 Text Label 6450 4100 0    50   ~ 0
 INPUT
+Text Label 7600 4500 0    50   ~ 0
+INPUT
+Text Label 6300 3950 0    50   ~ 0
+uCtoLED
+Text Label 6950 3750 3    50   ~ 0
+LEDtoR
+Wire Wire Line
+	5700 4800 5700 4700
+NoConn ~ 6300 4200
+NoConn ~ 5100 4000
+NoConn ~ 5100 4100
+NoConn ~ 5100 4200
+$Comp
+L power:PWR_FLAG #FLG01
+U 1 1 5D78C01A
+P 8450 5650
+F 0 "#FLG01" H 8450 5725 50  0001 C CNN
+F 1 "PWR_FLAG" H 8450 5824 50  0000 C CNN
+F 2 "" H 8450 5650 50  0001 C CNN
+F 3 "~" H 8450 5650 50  0001 C CNN
+	1    8450 5650
+	1    0    0    -1
+$EndComp
+$Comp
+L power:PWR_FLAG #FLG02
+U 1 1 5D78C036
+P 8900 5650
+F 0 "#FLG02" H 8900 5725 50  0001 C CNN
+F 1 "PWR_FLAG" H 8900 5824 50  0000 C CNN
+F 2 "" H 8900 5650 50  0001 C CNN
+F 3 "~" H 8900 5650 50  0001 C CNN
+	1    8900 5650
+	1    0    0    -1
+$EndComp
+$Comp
+L power:VCC #PWR06
+U 1 1 5D78C050
+P 8450 5800
+F 0 "#PWR06" H 8450 5650 50  0001 C CNN
+F 1 "VCC" H 8467 5973 50  0000 C CNN
+F 2 "" H 8450 5800 50  0001 C CNN
+F 3 "" H 8450 5800 50  0001 C CNN
+	1    8450 5800
+	-1   0    0    1
+$EndComp
+$Comp
+L power:GND #PWR07
+U 1 1 5D78C088
+P 8900 5800
+F 0 "#PWR07" H 8900 5550 50  0001 C CNN
+F 1 "GND" H 8905 5627 50  0000 C CNN
+F 2 "" H 8900 5800 50  0001 C CNN
+F 3 "" H 8900 5800 50  0001 C CNN
+	1    8900 5800
+	1    0    0    -1
+$EndComp
+Wire Wire Line
+	8450 5800 8450 5650
+Wire Wire Line
+	8900 5650 8900 5800
+Text Notes 8050 6250 0    50   ~ 0
+Needed to supress KiCad DRC warning.\n
+Wire Notes Line
+	7750 5300 7750 6350
+Wire Notes Line
+	7750 6350 9750 6350
+Wire Notes Line
+	9750 6350 9750 5300
+Wire Notes Line
+	9750 5300 7750 5300
+Wire Wire Line
+	5700 3500 5700 3400
 $EndSCHEMATC

Commit message: Made final changes to the board design and added screenshots of the board.
Signed-off-by: Suyash <in.suyash@gmail.com>
Other:
- moved on the sheet: D1, J1, R1, R2, U1
Changed lines of the file:
@@
 L microchip_pic12mcu:PIC12C508A-ISN U1
 U 1 1 5D761873
-P 5700 4100
-F 0 "U1" H 6050 4600 50  0000 C CNN
-F 1 "PIC12C508A-ISN" H 5300 4600 50  0000 C CNN
-F 2 "Package_DIP:DIP-8_W7.62mm" H 6300 4750 50  0001 C CNN
-F 3 "http://ww1.microchip.com/downloads/en/devicedoc/40139e.pdf" H 5700 4100 50  0001 C CNN
-	1    5700 4100
+P 4750 3550
+F 0 "U1" H 5100 4050 50  0000 C CNN
+F 1 "PIC12C508A-ISN" H 4350 4050 50  0000 C CNN
+F 2 "Package_DIP:DIP-8_W7.62mm" H 5350 4200 50  0001 C CNN
+F 3 "http://ww1.microchip.com/downloads/en/devicedoc/40139e.pdf" H 4750 3550 50  0001 C CNN
+	1    4750 3550
 	-1   0    0    -1
 $EndComp
@@
 L Device:LED D1
 U 1 1 5D761962
-P 6700 3750
-F 0 "D1" H 6691 3966 50  0000 C CNN
-F 1 "LED" H 6691 3875 50  0000 C CNN
-F 2 "LED_THT:LED_D5.0mm" H 6700 3750 50  0001 C CNN
-F 3 "~" H 6700 3750 50  0001 C CNN
-	1    6700 3750
+P 5750 3200
+F 0 "D1" H 5741 3416 50  0000 C CNN
+F 1 "LED" H 5741 3325 50  0000 C CNN
+F 2 "LED_THT:LED_D5.0mm" H 5750 3200 50  0001 C CNN
+F 3 "~" H 5750 3200 50  0001 C CNN
+	1    5750 3200
 	1    0    0    -1
 $EndComp
@@
 L myLib:MYCONN3 J1
 U 1 1 5D761E83
-P 6850 4500
-F 0 "J1" H 6856 4825 50  0000 C CNN
-F 1 "MYCONN3" H 6856 4734 50  0000 C CNN
-F 2 "Connector:Banana_Jack_3Pin" H 6950 4500 50  0001 C CNN
-F 3 "" H 6950 4500 50  0001 C CNN
-	1    6850 4500
+P 5900 3950
+F 0 "J1" H 5906 4275 50  0000 C CNN
+F 1 "MYCONN3" H 5906 4184 50  0000 C CNN
+F 2 "Connector:Banana_Jack_3Pin" H 6000 3950 50  0001 C CNN
+F 3 "" H 6000 3950 50  0001 C CNN
+	1    5900 3950
 	1    0    0    -1
 $EndComp
@@
 L power:VCC #PWR01
 U 1 1 5D761F83
-P 5700 3400
-F 0 "#PWR01" H 5700 3250 50  0001 C CNN
-F 1 "VCC" H 5717 3573 50  0000 C CNN
-F 2 "" H 5700 3400 50  0001 C CNN
-F 3 "" H 5700 3400 50  0001 C CNN
-	1    5700 3400
+P 4750 2850
+F 0 "#PWR01" H 4750 2700 50  0001 C CNN
+F 1 "VCC" H 4767 3023 50  0000 C CNN
+F 2 "" H 4750 2850 50  0001 C CNN
+F 3 "" H 4750 2850 50  0001 C CNN
+	1    4750 2850
 	1    0    0    -1
 $EndComp
@@
 L power:GND #PWR02
 U 1 1 5D761FCE
-P 5700 4800
-F 0 "#PWR02" H 5700 4550 50  0001 C CNN
-F 1 "GND" H 5705 4627 50  0000 C CNN
-F 2 "" H 5700 4800 50  0001 C CNN
-F 3 "" H 5700 4800 50  0001 C CNN
-	1    5700 4800
+P 4750 4250
+F 0 "#PWR02" H 4750 4000 50  0001 C CNN
+F 1 "GND" H 4755 4077 50  0000 C CNN
+F 2 "" H 4750 4250 50  0001 C CNN
+F 3 "" H 4750 4250 50  0001 C CNN
+	1    4750 4250
 	1    0    0    -1
 $EndComp
@@
 L Device:R R1
 U 1 1 5D762095
-P 7200 3750
-F 0 "R1" V 7300 3700 50  0000 L CNN
-F 1 "1 k" V 7100 3700 50  0000 L CNN
-F 2 "Resistor_THT:R_Axial_DIN0204_L3.6mm_D1.6mm_P7.62mm_Horizontal" V 7130 3750 50  0001 C CNN
-F 3 "~" H 7200 3750 50  0001 C CNN
-	1    7200 3750
+P 6250 3200
+F 0 "R1" V 6350 3150 50  0000 L CNN
+F 1 "1 k" V 6150 3150 50  0000 L CNN
+F 2 "Resistor_THT:R_Axial_DIN0204_L3.6mm_D1.6mm_P7.62mm_Horizontal" V 6180 3200 50  0001 C CNN
+F 3 "~" H 6250 3200 50  0001 C CNN
+	1    6250 3200
 	0    -1   -1   0
 $EndComp
@@
 L power:VCC #PWR05
 U 1 1 5D76212F
-P 7400 3550
-F 0 "#PWR05" H 7400 3400 50  0001 C CNN
-F 1 "VCC" H 7417 3723 50  0000 C CNN
-F 2 "" H 7400 3550 50  0001 C CNN
-F 3 "" H 7400 3550 50  0001 C CNN
-	1    7400 3550
+P 6450 3000
+F 0 "#PWR05" H 6450 2850 50  0001 C CNN
+F 1 "VCC" H 6467 3173 50  0000 C CNN
+F 2 "" H 6450 3000 50  0001 C CNN
+F 3 "" H 6450 3000 50  0001 C CNN
+	1    6450 3000
 	1    0    0    -1
 $EndComp
@@
 L Device:R R2
 U 1 1 5D7624C6
-P 7350 4500
-F 0 "R2" V 7450 4450 50  0000 L CNN
-F 1 "100R" V 7250 4450 50  0000 L CNN
-F 2 "Resistor_THT:R_Axial_DIN0204_L3.6mm_D1.6mm_P7.62mm_Horizontal" V 7280 4500 50  0001 C CNN
-F 3 "~" H 7350 4500 50  0001 C CNN
-	1    7350 4500
+P 6400 3950
+F 0 "R2" V 6500 3900 50  0000 L CNN
+F 1 "100R" V 6300 3900 50  0000 L CNN
+F 2 "Resistor_THT:R_Axial_DIN0204_L3.6mm_D1.6mm_P7.62mm_Horizontal" V 6330 3950 50  0001 C CNN
+F 3 "~" H 6400 3950 50  0001 C CNN
+	1    6400 3950
 	0    -1   -1   0
 $EndComp
 Wire Wire Line
-	6300 4000 6300 3750
-Wire Wire Line
-	6300 3750 6550 3750
-Wire Wire Line
-	6850 3750 7050 3750
-Wire Wire Line
-	7350 3750 7400 3750
-Wire Wire Line
-	7400 3750 7400 3550
+	5350 3450 5350 3200
+Wire Wire Line
+	5350 3200 5600 3200
+Wire Wire Line
+	5900 3200 6100 3200
+Wire Wire Line
+	6400 3200 6450 3200
+Wire Wire Line
+	6450 3200 6450 3000
 $Comp
 L power:VCC #PWR03
 U 1 1 5D7625C1
-P 7150 4250
-F 0 "#PWR03" H 7150 4100 50  0001 C CNN
-F 1 "VCC" H 7167 4423 50  0000 C CNN
-F 2 "" H 7150 4250 50  0001 C CNN
-F 3 "" H 7150 4250 50  0001 C CNN
-	1    7150 4250
+P 6200 3700
+F 0 "#PWR03" H 6200 3550 50  0001 C CNN
+F 1 "VCC" H 6217 3873 50  0000 C CNN
+F 2 "" H 6200 3700 50  0001 C CNN
+F 3 "" H 6200 3700 50  0001 C CNN
+	1    6200 3700
 	1    0    0    -1
 $EndComp
@@
 L power:GND #PWR04
 U 1 1 5D762617
-P 7150 4700
-F 0 "#PWR04" H 7150 4450 50  0001 C CNN
-F 1 "GND" H 7155 4527 50  0000 C CNN
-F 2 "" H 7150 4700 50  0001 C CNN
-F 3 "" H 7150 4700 50  0001 C CNN
-	1    7150 4700
-	1    0    0    -1
-$EndComp
-Wire Wire Line
-	7050 4400 7150 4400
-Wire Wire Line
-	7150 4400 7150 4250
-Wire Wire Line
-	7050 4600 7150 4600
-Wire Wire Line
-	7150 4600 7150 4700
-Wire Wire Line
-	7050 4500 7200 4500
-Wire Wire Line
-	7500 4500 7700 4500
-Wire Wire Line
-	6300 4100 6700 4100
-Text Label 6450 4100 0    50   ~ 0
+P 6200 4150
+F 0 "#PWR04" H 6200 3900 50  0001 C CNN
+F 1 "GND" H 6205 3977 50  0000 C CNN
+F 2 "" H 6200 4150 50  0001 C CNN
+F 3 "" H 6200 4150 50  0001 C CNN
+	1    6200 4150
+	1    0    0    -1
+$EndComp
+Wire Wire Line
+	6100 3850 6200 3850
+Wire Wire Line
+	6200 3850 6200 3700
+Wire Wire Line
+	6100 4050 6200 4050
+Wire Wire Line
+	6200 4050 6200 4150
+Wire Wire Line
+	6100 3950 6250 3950
+Wire Wire Line
+	6550 3950 6750 3950
+Wire Wire Line
+	5350 3550 5750 3550
+Text Label 5500 3550 0    50   ~ 0
 INPUT
-Text Label 7600 4500 0    50   ~ 0
+Text Label 6650 3950 0    50   ~ 0
 INPUT
-Text Label 6300 3950 0    50   ~ 0
+Text Label 5350 3400 0    50   ~ 0
 uCtoLED
-Text Label 6950 3750 3    50   ~ 0
+Text Label 6000 3200 3    50   ~ 0
 LEDtoR
 Wire Wire Line
-	5700 4800 5700 4700
-NoConn ~ 6300 4200
-NoConn ~ 5100 4000
-NoConn ~ 5100 4100
-NoConn ~ 5100 4200
+	4750 4250 4750 4150
+NoConn ~ 5350 3650
+NoConn ~ 4150 3450
+NoConn ~ 4150 3550
+NoConn ~ 4150 3650
 $Comp
 L power:PWR_FLAG #FLG01
 U 1 1 5D78C01A
-P 8450 5650
-F 0 "#FLG01" H 8450 5725 50  0001 C CNN
-F 1 "PWR_FLAG" H 8450 5824 50  0000 C CNN
-F 2 "" H 8450 5650 50  0001 C CNN
-F 3 "~" H 8450 5650 50  0001 C CNN
-	1    8450 5650
+P 9150 3400
+F 0 "#FLG01" H 9150 3475 50  0001 C CNN
+F 1 "PWR_FLAG" H 9150 3574 50  0000 C CNN
+F 2 "" H 9150 3400 50  0001 C CNN
+F 3 "~" H 9150 3400 50  0001 C CNN
+	1    9150 3400
 	1    0    0    -1
 $EndComp
@@
 L power:PWR_FLAG #FLG02
 U 1 1 5D78C036
-P 8900 5650
-F 0 "#FLG02" H 8900 5725 50  0001 C CNN
-F 1 "PWR_FLAG" H 8900 5824 50  0000 C CNN
-F 2 "" H 8900 5650 50  0001 C CNN
-F 3 "~" H 8900 5650 50  0001 C CNN
-	1    8900 5650
+P 9600 3400
+F 0 "#FLG02" H 9600 3475 50  0001 C CNN
+F 1 "PWR_FLAG" H 9600 3574 50  0000 C CNN
+F 2 "" H 9600 3400 50  0001 C CNN
+F 3 "~" H 9600 3400 50  0001 C CNN
+	1    9600 3400
 	1    0    0    -1
 $EndComp
@@
 L power:VCC #PWR06
 U 1 1 5D78C050
-P 8450 5800
-F 0 "#PWR06" H 8450 5650 50  0001 C CNN
-F 1 "VCC" H 8467 5973 50  0000 C CNN
-F 2 "" H 8450 5800 50  0001 C CNN
-F 3 "" H 8450 5800 50  0001 C CNN
-	1    8450 5800
+P 9150 3550
+F 0 "#PWR06" H 9150 3400 50  0001 C CNN
+F 1 "VCC" H 9167 3723 50  0000 C CNN
+F 2 "" H 9150 3550 50  0001 C CNN
+F 3 "" H 9150 3550 50  0001 C CNN
+	1    9150 3550
 	-1   0    0    1
 $EndComp
@@
 L power:GND #PWR07
 U 1 1 5D78C088
-P 8900 5800
-F 0 "#PWR07" H 8900 5550 50  0001 C CNN
-F 1 "GND" H 8905 5627 50  0000 C CNN
-F 2 "" H 8900 5800 50  0001 C CNN
-F 3 "" H 8900 5800 50  0001 C CNN
-	1    8900 5800
-	1    0    0    -1
-$EndComp
-Wire Wire Line
-	8450 5800 8450 5650
-Wire Wire Line
-	8900 5650 8900 5800
-Text Notes 8050 6250 0    50   ~ 0
+P 9600 3550
+F 0 "#PWR07" H 9600 3300 50  0001 C CNN
+F 1 "GND" H 9605 3377 50  0000 C CNN
+F 2 "" H 9600 3550 50  0001 C CNN
+F 3 "" H 9600 3550 50  0001 C CNN
+	1    9600 3550
+	1    0    0    -1
+$EndComp
+Wire Wire Line
+	9150 3550 9150 3400
+Wire Wire Line
+	9600 3400 9600 3550
+Text Notes 8750 4000 0    50   ~ 0
 Needed to supress KiCad DRC warning.\n
-Wire Notes Line
-	7750 5300 7750 6350
-Wire Notes Line
-	7750 6350 9750 6350
-Wire Notes Line
-	9750 6350 9750 5300
-Wire Notes Line
-	9750 5300 7750 5300
-Wire Wire Line
-	5700 3500 5700 3400
+Wire Wire Line
+	4750 2950 4750 2850
 $EndSCHEMATC
